File: BedoPadPcb.sch (KiCad schematic (older format))
At the start: 37 parts

Commit message: Pcb layout finished
Parts:
- removed U?: ProMicro, symbol promicro:ProMicro
- added H1, H2: MountingHole_Pad, kbd:1pin_conn, symbol Mechanical:MountingHole_Pad
- added OL1: OLED, kbd:OLED_v2, symbol kbd:OLED
- added U1: ProMicro, kbd:ProMicro_v3, symbol kbd:ProMicro
- D1, D10, D11, D12, D13, D14, D15, D16, D17, D18, D2, D3, D4, D5, D6, D7, D8, D9: renamed from D?; footprint (none) -> kbd:D3_TH
- SW1: renamed from SW?; footprint (none) -> Keebio-Parts:RotaryEncoder_EC11
- SW10, SW11, SW12, SW13, SW14, SW15, SW16, SW17, SW18, SW2, SW3, SW4, SW5, SW6, SW7, SW8, SW9: renamed from SW?; footprint (none) -> kbd:CherryMX_Hotswap
Connections:
- net Col0: now also U1.7 (4/D4)
- net Col1: now also U1.15 (B3/14)
- net Col2: now also U1.14 (B2/16)
- net Col3: now also U1.13 (B6/10)
- net EncoderGND: now also U1.3 (GND)
- net EncoderPadA: now also U1.10 (7/E6)
- net EncoderPadB: now also U1.11 (8/B4)
- net Row0: now also D14.1 (K), D4.1 (K), D9.1 (K), U1.20 (F4/A3); no longer D14.2 (A), D4.2 (A), D9.2 (A)
- net Row1: now also D10.1 (K), D15.1 (K), D5.1 (K), U1.19 (F5/A2); no longer D10.2 (A), D15.2 (A), D5.2 (A)
- net Row2: now also D1.1 (K), D11.1 (K), D16.1 (K), D6.1 (K), U1.18 (F6/A1); no longer D1.2 (A), D11.2 (A), D16.2 (A), D6.2 (A)
- net Row3: now also D12.1 (K), D17.1 (K), D2.1 (K), D7.1 (K), U1.17 (F7/A0); no longer D12.2 (A), D17.2 (A), D2.2 (A), D7.2 (A)
- net Row4: now also D13.1 (K), D18.1 (K), D3.1 (K), D8.1 (K), U1.16 (B1/15); no longer D13.2 (A), D18.2 (A), D3.2 (A), D8.2 (A)
- net at SW4.2: now also D4.2 (A); no longer D4.1 (K)
- net at SW9.2: now also D9.2 (A); no longer D9.1 (K)
- net at SW14.2: now also D14.2 (A); no longer D14.1 (K)
- net at SW5.2: now also D5.2 (A); no longer D5.1 (K)
- net at SW10.2: now also D10.2 (A); no longer D10.1 (K)
- net at SW15.2: now also D15.2 (A); no longer D15.1 (K)
- net at SW16.2: now also D16.2 (A); no longer D16.1 (K)
- net at SW11.2: now also D11.2 (A); no longer D11.1 (K)
- net at SW6.2: now also D6.2 (A); no longer D6.1 (K)
- net at SW7.2: now also D7.2 (A); no longer D7.1 (K)
- net at SW12.2: now also D12.2 (A); no longer D12.1 (K)
- net at SW17.2: now also D17.2 (A); no longer D17.1 (K)
- net at SW8.2: now also D8.2 (A); no longer D8.1 (K)
- net at SW13.2: now also D13.2 (A); no longer D13.1 (K)
- net at SW18.2: now also D18.2 (A); no longer D18.1 (K)
- net at SW2.2: now also D2.2 (A); no longer D2.1 (K)
- net at SW3.2: now also D3.2 (A); no longer D3.1 (K)
- net at SW1.S2: now also D1.2 (A); no longer D1.1 (K)
- new net OledGND: OL1.4 (GND), U1.4 (GND)
- new net OledSCL: OL1.2 (SCL), U1.6 (3/D0/SCL)
- new net OledSDA: OL1.1 (SDA), U1.5 (2/D1/SDA)
- new net OledVCC: OL1.3 (VCC), U1.21 (VCC)
- new net ResetVIA1: H1.1, U1.23 (GND)
- new net ResetVIA2: H2.1, U1.22 (RST)
