File: PCB/BedoPadPcb.kicad_pcb (KiCad board)
At the start: 2 copper layers, 127 x 106.4 mm, 40 parts, among them SW1 Rotary_Encoder_Switch, SW10 CherryMX, SW11 CherryMX, SW12 CherryMX, SW13 CherryMX, SW14 CherryMX, SW15 CherryMX, SW16 CherryMX, SW17 CherryMX, SW18 CherryMX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

Commit message: Restructure
Parts:
- added G***: LOGO, bedodev:bedodev_logo, B.Cu at (31.1, 85.5)
Routing:
- net Row3: track 0.00 -> 226.8 mm
- net Row4: track 0.00 -> 219.6 mm
- net Col3: track 0.00 -> 210.2 mm
- net Col2: track 0.00 -> 192.1 mm
- net Row2: track 0.00 -> 190.1 mm
- net Col1: track 0.00 -> 157.2 mm
- net Col0: track 0.00 -> 129.9 mm
- net Row1: track 0.00 -> 93.9 mm
- net Row0: track 0.00 -> 87.3 mm
- net EncoderGND: track 0.00 -> 51.0 mm
- net EncoderPadB: track 0.00 -> 34.4 mm
- net EncoderPadA: track 0.00 -> 30.1 mm
- net OledGND: track 0.00 -> 29.9 mm
- net ResetVIA1: track 0.00 -> 29.8 mm
- net ResetVIA2: track 0.00 -> 29.7 mm
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Other:
- board size 127 x 106.4 mm -> 127 x 101.6 mm
- board text added: "BedoPad MK1"
- board text added: "GND"
- board text added: "Prototype 1"
- board text added: "RESET"

Commit message: Final PCB
Parts:
- added G***: LOGO, bedodev:bedodev_logo_japanese, B.Cu at (149.2, 61.2)
- added G***: LOGO, bedodev:bedodev_logo_japanese, F.Cu at (36.5, 149.2)
- added REF**: OSHW-Symbol_6.7x6mm_SilkScreen, Symbol:OSHW-Symbol_6.7x6mm_SilkScreen, B.Cu at (141.2, 147.4)
- added REF**: M2_Hole_TH, kbd:M2_Hole_TH, F.Cu at (70.3, 99.1)
- added REF**: M2_Hole_TH, kbd:M2_Hole_TH, F.Cu at (147.6, 147.6)
- added REF**: M2_Hole_TH, kbd:M2_Hole_TH, F.Cu at (27.0, 147.6)
- added REF**: M2_Hole_TH, kbd:M2_Hole_TH, F.Cu at (27.0, 52.4)
- added REF**: M2_Hole_TH, kbd:M2_Hole_TH, F.Cu at (147.6, 52.4)
- D1, D10, D11, D12, D13, D14, D15, D16, D17, D18, D2, D3, D4, D5, D6, D7, D8, D9: footprint kbd:D3_TH -> Keebio-Parts:Diode
- turned D1 to 270 degrees
- turned D10 to 270 degrees
- turned D11 to 270 degrees
- turned D12 to 270 degrees
- turned D13 to 270 degrees
- turned D14 to 270 degrees
- turned D15 to 270 degrees
- turned D16 to 270 degrees
- turned D17 to 270 degrees
- turned D18 to 270 degrees
- turned D2 to 270 degrees
- turned D3 to 270 degrees
- turned D4 to 270 degrees
- turned D5 to 270 degrees
- turned D6 to 270 degrees
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Connections:
- D1 pad 1: Row2 -> Net-(D1-Pad1)
- D1 pad 2: Net-(D1-Pad2) -> Row2
- D10 pad 1: Row1 -> Net-(D10-Pad1)
- D10 pad 2: Net-(D10-Pad2) -> Row1
- D11 pad 1: Row2 -> Net-(D11-Pad1)
- D11 pad 2: Net-(D11-Pad2) -> Row2
- D12 pad 1: Row3 -> Net-(D12-Pad1)
- D12 pad 2: Net-(D12-Pad2) -> Row3
- D13 pad 1: Row4 -> Net-(D13-Pad1)
- D13 pad 2: Net-(D13-Pad2) -> Row4
- D14 pad 1: Row0 -> Net-(D14-Pad1)
- D14 pad 2: Net-(D14-Pad2) -> Row0
- D15 pad 1: Row1 -> Net-(D15-Pad1)
- D15 pad 2: Net-(D15-Pad2) -> Row1
- D16 pad 1: Row2 -> Net-(D16-Pad1)
- D16 pad 2: Net-(D16-Pad2) -> Row2
- D17 pad 1: Row3 -> Net-(D17-Pad1)
- D17 pad 2: Net-(D17-Pad2) -> Row3
- D18 pad 1: Row4 -> Net-(D18-Pad1)
- D18 pad 2: Net-(D18-Pad2) -> Row4
- D2 pad 1: Row3 -> Net-(D2-Pad1)
- D2 pad 2: Net-(D2-Pad2) -> Row3
- D3 pad 1: Row4 -> Net-(D3-Pad1)
- D3 pad 2: Net-(D3-Pad2) -> Row4
- D4 pad 1: Row0 -> Net-(D4-Pad1)
- D4 pad 2: Net-(D4-Pad2) -> Row0
- D5 pad 1: Row1 -> Net-(D5-Pad1)
- D5 pad 2: Net-(D5-Pad2) -> Row1
- D6 pad 1: Row2 -> Net-(D6-Pad1)
- D6 pad 2: Net-(D6-Pad2) -> Row2
- D7 pad 1: Row3 -> Net-(D7-Pad1)
- D7 pad 2: Net-(D7-Pad2) -> Row3
- D8 pad 1: Row4 -> Net-(D8-Pad1)
- D8 pad 2: Net-(D8-Pad2) -> Row4
- D9 pad 1: Row0 -> Net-(D9-Pad1)
- D9 pad 2: Net-(D9-Pad2) -> Row0
- SW1 pad S2: Net-(D1-Pad2) -> Net-(D1-Pad1)
- SW10 pad 2: Net-(D10-Pad2) -> Net-(D10-Pad1)
- SW11 pad 2: Net-(D11-Pad2) -> Net-(D11-Pad1)
- SW12 pad 2: Net-(D12-Pad2) -> Net-(D12-Pad1)
- SW13 pad 2: Net-(D13-Pad2) -> Net-(D13-Pad1)
- SW14 pad 2: Net-(D14-Pad2) -> Net-(D14-Pad1)
- SW15 pad 2: Net-(D15-Pad2) -> Net-(D15-Pad1)
- SW16 pad 2: Net-(D16-Pad2) -> Net-(D16-Pad1)
- SW17 pad 2: Net-(D17-Pad2) -> Net-(D17-Pad1)
- SW18 pad 2: Net-(D18-Pad2) -> Net-(D18-Pad1)
- SW2 pad 2: Net-(D2-Pad2) -> Net-(D2-Pad1)
- SW3 pad 2: Net-(D3-Pad2) -> Net-(D3-Pad1)
- SW4 pad 2: Net-(D4-Pad2) -> Net-(D4-Pad1)
- SW5 pad 2: Net-(D5-Pad2) -> Net-(D5-Pad1)
- SW6 pad 2: Net-(D6-Pad2) -> Net-(D6-Pad1)
- SW7 pad 2: Net-(D7-Pad2) -> Net-(D7-Pad1)
- SW8 pad 2: Net-(D8-Pad2) -> Net-(D8-Pad1)
- SW9 pad 2: Net-(D9-Pad2) -> Net-(D9-Pad1)
Routing:
- net Net-(D1-Pad2): track 5.36 -> 0.00 mm
- net Net-(D1-Pad1): track 0.00 -> 5.02 mm
- net Net-(D9-Pad2): track 4.08 -> 0.00 mm
- net Net-(D8-Pad2): track 4.08 -> 0.00 mm
- net Net-(D7-Pad2): track 4.08 -> 0.00 mm
- net Net-(D6-Pad2): track 4.08 -> 0.00 mm
- net Net-(D5-Pad2): track 4.08 -> 0.00 mm
- net Net-(D4-Pad2): track 4.08 -> 0.00 mm
- net Net-(D3-Pad2): track 4.08 -> 0.00 mm
- net Net-(D2-Pad2): track 4.08 -> 0.00 mm
- net Net-(D18-Pad2): track 4.08 -> 0.00 mm
- net Net-(D17-Pad2): track 4.08 -> 0.00 mm
- net Net-(D16-Pad2): track 4.08 -> 0.00 mm
- net Net-(D15-Pad2): track 4.08 -> 0.00 mm
- net Net-(D14-Pad2): track 4.08 -> 0.00 mm
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Other:
- board text removed: "Prototype 1"
