File: PCB/BedoPadPcb.sch (KiCad schematic (older format))
At the start: 40 parts, among them SW1 Rotary_Encoder_Switch, SW10 CherryMX, SW11 CherryMX, SW12 CherryMX, SW13 CherryMX, SW14 CherryMX, SW15 CherryMX, SW16 CherryMX, SW17 CherryMX, SW18 CherryMX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

Commit message: Final PCB
Connections:
- net Row0: now also D14.2 (A), D4.2 (A), D9.2 (A); no longer D14.1 (K), D4.1 (K), D9.1 (K)
- net Row1: now also D10.2 (A), D15.2 (A), D5.2 (A); no longer D10.1 (K), D15.1 (K), D5.1 (K)
- net Row2: now also D1.2 (A), D11.2 (A), D16.2 (A), D6.2 (A); no longer D1.1 (K), D11.1 (K), D16.1 (K), D6.1 (K)
- net Row3: now also D12.2 (A), D17.2 (A), D2.2 (A), D7.2 (A); no longer D12.1 (K), D17.1 (K), D2.1 (K), D7.1 (K)
- net Row4: now also D13.2 (A), D18.2 (A), D3.2 (A), D8.2 (A); no longer D13.1 (K), D18.1 (K), D3.1 (K), D8.1 (K)
- net at SW4.2: now also D4.1 (K); no longer D4.2 (A)
- net at SW9.2: now also D9.1 (K); no longer D9.2 (A)
- net at SW14.2: now also D14.1 (K); no longer D14.2 (A)
- net at SW5.2: now also D5.1 (K); no longer D5.2 (A)
- net at SW10.2: now also D10.1 (K); no longer D10.2 (A)
- net at SW15.2: now also D15.1 (K); no longer D15.2 (A)
- net at SW16.2: now also D16.1 (K); no longer D16.2 (A)
- net at SW11.2: now also D11.1 (K); no longer D11.2 (A)
- net at SW6.2: now also D6.1 (K); no longer D6.2 (A)
- net at SW7.2: now also D7.1 (K); no longer D7.2 (A)
- net at SW12.2: now also D12.1 (K); no longer D12.2 (A)
- net at SW17.2: now also D17.1 (K); no longer D17.2 (A)
- net at SW8.2: now also D8.1 (K); no longer D8.2 (A)
- net at SW13.2: now also D13.1 (K); no longer D13.2 (A)
- net at SW18.2: now also D18.1 (K); no longer D18.2 (A)
- net at SW2.2: now also D2.1 (K); no longer D2.2 (A)
- net at SW3.2: now also D3.1 (K); no longer D3.2 (A)
- net at SW1.S2: now also D1.1 (K); no longer D1.2 (A)
Changed lines of the file:
@@
 F 3 "~" H 2500 3650 50  0001 C CNN
 	1    2500 3650
-	0    -1   -1   0
+	0    1    1    0
 $EndComp
 $Comp
@@
 F 3 "~" H 2500 4450 50  0001 C CNN
 	1    2500 4450
-	0    -1   -1   0
+	0    1    1    0
 $EndComp
 $Comp
@@
 F 3 "~" H 3850 5000 50  0001 C CNN
 	1    3850 5000
-	0    -1   -1   0
+	0    1    1    0
 $EndComp
 $Comp
@@
 F 3 "~" H 4600 5000 50  0001 C CNN
 	1    4600 5000
-	0    -1   -1   0
+	0    1    1    0
 $EndComp
 $Comp
@@
 F 3 "~" H 5300 5000 50  0001 C CNN
 	1    5300 5000
-	0    -1   -1   0
+	0    1    1    0
 $EndComp
 $Comp
@@
 F 3 "~" H 5300 4000 50  0001 C CNN
 	1    5300 4000
-	0    -1   -1   0
+	0    1    1    0
 $EndComp
 $Comp
@@
 F 3 "~" H 4600 4000 50  0001 C CNN
 	1    4600 4000
-	0    -1   -1   0
+	0    1    1    0
 $EndComp
 $Comp
@@
 F 3 "~" H 3850 4000 50  0001 C CNN
 	1    3850 4000
-	0    -1   -1   0
+	0    1    1    0
 $EndComp
 $Comp
@@
 F 3 "~" H 5300 3100 50  0001 C CNN
 	1    5300 3100
-	0    -1   -1   0
+	0    1    1    0
 $EndComp
 $Comp
@@
 F 3 "~" H 4600 3100 50  0001 C CNN
 	1    4600 3100
-	0    -1   -1   0
+	0    1    1    0
 $EndComp
 $Comp
@@
 F 3 "~" H 3850 3100 50  0001 C CNN
 	1    3850 3100
-	0    -1   -1   0
+	0    1    1    0
 $EndComp
 $Comp
@@
 F 3 "~" H 5300 2200 50  0001 C CNN
 	1    5300 2200
-	0    -1   -1   0
+	0    1    1    0
 $EndComp
 $Comp
@@
 F 3 "~" H 4600 2200 50  0001 C CNN
 	1    4600 2200
-	0    -1   -1   0
+	0    1    1    0
 $EndComp
 $Comp
@@
 F 3 "~" H 3850 2200 50  0001 C CNN
 	1    3850 2200
-	0    -1   -1   0
+	0    1    1    0
 $EndComp
 $Comp
@@
 F 3 "~" H 5300 1300 50  0001 C CNN
 	1    5300 1300
-	0    -1   -1   0
+	0    1    1    0
 $EndComp
 $Comp
@@
 F 3 "~" H 4600 1300 50  0001 C CNN
 	1    4600 1300
-	0    -1   -1   0
+	0    1    1    0
 $EndComp
 $Comp
@@
 F 3 "~" H 3850 1300 50  0001 C CNN
 	1    3850 1300
-	0    -1   -1   0
+	0    1    1    0
 $EndComp
 Wire Wire Line
@@
 F 3 "~" H 1850 2250 50  0001 C CNN
 	1    1850 2250
-	0    -1   -1   0
+	0    1    1    0
 $EndComp
 Wire Wire Line
@@
 	-1   0    0    -1
 $EndComp
-Wire Wire Line
-	1850 3300 3850 3300
-Connection ~ 3850 3300
-Wire Wire Line
-	2500 4200 3850 4200
-Connection ~ 3850 4200
-Wire Wire Line
-	2500 5200 3850 5200
-Connection ~ 3850 5200
-Wire Wire Line
-	3850 5200 4600 5200
-Connection ~ 4600 5200
-Wire Wire Line
-	4600 5200 5300 5200
-Connection ~ 5300 5200
-Wire Wire Line
-	5300 5200 5950 5200
-Wire Wire Line
-	3850 4200 4600 4200
-Connection ~ 4600 4200
-Wire Wire Line
-	4600 4200 5300 4200
-Connection ~ 5300 4200
-Wire Wire Line
-	5300 4200 5950 4200
-Connection ~ 5300 3300
-Wire Wire Line
-	5300 3300 5950 3300
-Wire Wire Line
-	3850 3300 4600 3300
-Connection ~ 4600 3300
-Wire Wire Line
-	4600 3300 5300 3300
-Wire Wire Line
-	3850 2400 4600 2400
-Connection ~ 4600 2400
-Wire Wire Line
-	4600 2400 5300 2400
-Connection ~ 5300 2400
-Wire Wire Line
-	5300 2400 5950 2400
-Wire Wire Line
-	3850 1500 4600 1500
-Connection ~ 4600 1500
-Wire Wire Line
-	4600 1500 5300 1500
-Connection ~ 5300 1500
-Wire Wire Line
-	5300 1500 5950 1500
 Text GLabel 9050 1350 0    50   Input ~ 0
 ResetVIA1
@@
 	1    0    0    -1
 $EndComp
+Wire Wire Line
+	2500 4200 3850 4200
+Connection ~ 3850 4200
+Wire Wire Line
+	2500 5200 3850 5200
+Connection ~ 3850 5200
+Wire Wire Line
+	3850 5200 4600 5200
+Connection ~ 4600 5200
+Wire Wire Line
+	4600 5200 5300 5200
+Connection ~ 5300 5200
+Wire Wire Line
+	5300 5200 5950 5200
+Connection ~ 5300 4200
+Wire Wire Line
+	5300 4200 5950 4200
+Wire Wire Line
+	3850 4200 4600 4200
+Connection ~ 4600 4200
+Wire Wire Line
+	4600 4200 5300 4200
+Wire Wire Line
+	1850 3300 3850 3300
+Connection ~ 3850 3300
+Wire Wire Line
+	3850 3300 4600 3300
+Connection ~ 4600 3300
+Wire Wire Line
+	4600 3300 5300 3300
+Connection ~ 5300 3300
+Wire Wire Line
+	5300 3300 5950 3300
+Connection ~ 5300 2400
+Wire Wire Line
+	5300 2400 5950 2400
+Wire Wire Line
+	3850 2400 4600 2400
+Connection ~ 4600 2400
+Wire Wire Line
+	4600 2400 5300 2400
+Wire Wire Line
+	3850 1500 4600 1500
+Connection ~ 4600 1500
+Wire Wire Line
+	4600 1500 5300 1500
+Connection ~ 5300 1500
+Wire Wire Line
+	5300 1500 5950 1500
 $EndSCHEMATC
